Commit message: Consistency between different xml declarations

File: gazebo_plugins/test/multi_robot_scenario/xacro/camera/camera.xacro (robot description, xacro)
@@ -1,4 +1,4 @@
 <?xml version="1.0"?>
-<robot xmlns:xacro="http://www.ros.org/wiki/xacro">
+<robot xmlns:xacro="http://ros.org/wiki/xacro">
 <!-- Camera -->
 <xacro:macro name="cam" params="name parent xyz rpy">

File: gazebo_plugins/test/multi_robot_scenario/xacro/laser/hokuyo.xacro (robot description, xacro)
@@ -1,4 +1,4 @@
 <?xml version="1.0"?>
-<robot xmlns:xacro="http://www.ros.org/wiki/xacro">
+<robot xmlns:xacro="http://ros.org/wiki/xacro">
 <!-- Front Laser -->
 <xacro:macro name="laser" params="name parent xyz rpy meshes" >

File: gazebo_plugins/test/multi_robot_scenario/xacro/laser/hokuyo_gpu.xacro (robot description, xacro)
@@ -1,4 +1,4 @@
 <?xml version="1.0"?>
-<robot xmlns:xacro="http://www.ros.org/wiki/xacro">
+<robot xmlns:xacro="http://ros.org/wiki/xacro">
 <!-- Front Laser -->
 <xacro:macro name="laser_gpu" params="name parent xyz rpy meshes" >

File: gazebo_plugins/test/multi_robot_scenario/xacro/p3dx/pioneer3dx.xacro (robot description, xacro)
@@ -1,4 +1,4 @@
 <?xml version="1.0"?>
-<robot xmlns:xacro="http://www.ros.org/wiki/xacro" name="pioneer3dx" >
+<robot xmlns:xacro="http://ros.org/wiki/xacro" name="pioneer3dx" >
   <!-- Import Rviz colors -->
   <xacro:include filename="$(find gazebo_plugins)/test/multi_robot_scenario/xacro/materials.xacro" />

File: gazebo_plugins/test/multi_robot_scenario/xacro/p3dx/pioneer3dx_body.xacro (robot description, xacro)
@@ -1,4 +1,4 @@
 <?xml version="1.0"?>
-<robot xmlns:xacro="http://www.ros.org/wiki/xacro">
+<robot xmlns:xacro="http://ros.org/wiki/xacro">
   <xacro:include filename="inertia_tensors.xacro"/>
   <xacro:include filename="pioneer3dx_chassis.xacro"/>

File: gazebo_plugins/test/multi_robot_scenario/xacro/p3dx/pioneer3dx_plugins.xacro (robot description, xacro)
@@ -1,4 +1,4 @@
 <?xml version="1.0"?>
-<robot xmlns:xacro="http://www.ros.org/wiki/xacro">
+<robot xmlns:xacro="http://ros.org/wiki/xacro">
   <xacro:macro name="pioneer3dx_joints_state_publisher">
     <gazebo>

File: gazebo_plugins/test/tricycle_drive/xacro/tricycle/tricycle.xacro (robot description, xacro)
@@ -1,4 +1,4 @@
 <?xml version="1.0"?>
-<robot xmlns:xacro="http://www.ros.org/wiki/xacro" name="tricycle" >
+<robot xmlns:xacro="http://ros.org/wiki/xacro" name="tricycle" >
   <!-- Import Rviz colors -->
   <xacro:include filename="$(find gazebo_plugins)/test/tricycle_drive/xacro/materials.xacro" />

File: gazebo_plugins/test/tricycle_drive/xacro/tricycle/tricycle_body.xacro (robot description, xacro)
@@ -1,7 +1,7 @@
 <?xml version="1.0"?>
-<robot xmlns:xacro="http://www.ros.org/wiki/xacro">
-  <property name="M_PI" value="3.1415926535897931" />
-  <property name="radius_actuated_wheel" value="0.135" />
-  <property name="radius_encoder_wheel" value="0.135" />
+<robot xmlns:xacro="http://ros.org/wiki/xacro">
+  <xacro:property name="M_PI" value="3.1415926535897931" />
+  <xacro:property name="radius_actuated_wheel" value="0.135" />
+  <xacro:property name="radius_encoder_wheel" value="0.135" />
   <xacro:include filename="inertia_tensors.xacro"/>
   <xacro:include filename="tricycle_chassis.xacro"/>

File: gazebo_plugins/test/tricycle_drive/xacro/tricycle/tricycle_plugins.xacro (robot description, xacro)
@@ -1,4 +1,4 @@
 <?xml version="1.0"?>
-<robot xmlns:xacro="http://www.ros.org/wiki/xacro">
+<robot xmlns:xacro="http://ros.org/wiki/xacro">
   <xacro:macro name="tricycle_drive">
     <gazebo>
